File: boards/eos/eos-esp32-devkit/hardware/eos-esp32-devkit.kicad_sch (KiCad schematic)
At the start: 36 parts, among them J1 USB-C, J2 J2, J3 J3, Q1 MMBT3904, Q2 MMBT3904, SW1 EN, SW2 BOOT, U1 ESP32-WROOM-32E-N4, U2 USBLC6-2SC6, U3 AP7361C-33, U4 CP2102N-A02-GQFN24

Commit message: fix(boards): SP0503BAHTG ESD on EoS ESP32 DevKit; footprint BOM flag follows its symbol
- EoS ESP32 DevKit: the USBLC6-2SC6 is replaced with a Littelfuse SP0503BAHTG.
  - The USBLC6's data-line diodes run to its VBUS pin. After a host unplugs, the CP2102N's
    still-live D+ pull-up (the board can run from its 5V pin) would hold VBUS near 2 V, between
    the CP2102N VBUS pin's low and high thresholds (Table 3.7), so the bridge might never see the
    unplug.
  - The SP0503BAHTG is three diodes to ground with no path between the lines. It is the part the
    CP2102N data sheet shows on its USB pins (Figure 2.5).
  - D- goes on the pad nearer the connector, so the pair reaches the CP2102N (D+ above D-)
    without crossing.
  - Rebuilt: ERC 0, DRC errors 0, unconnected 0, parity 0, 8 silkscreen-at-edge warnings.
- tools/eos_boards: each footprint's "exclude from BOM" now follows its symbol's in_bom, as
  KiCad's Update PCB from Schematic does. A library test point otherwise excludes itself while
  its symbol counts it, and parity reports the mismatch. Tested in SpecTest.
Parts:
- U2: value USBLC6-2SC6 -> SP0503BAHTG; footprint Package_TO_SOT_SMD:SOT-23-6 -> Package_TO_SOT_SMD:SOT-143; symbol Power_Protection:USBLC6-2SC6 -> Power_Protection:SP0503BAHT; MPN USBLC6-2SC6 -> SP0503BAHTG; Manufacturer STMicroelectronics -> Littelfuse
Connections:
- net GND: now also U2.1 (A); no longer U2.2 (GND)
- net USB_D+: now also U2.3 (K); no longer U2.1 (I/O1), U2.6 (I/O1)
- net USB_D-: now also U2.2 (K); no longer U2.3 (I/O2), U2.4 (I/O2)
- net VBUS: now also U2.4 (K); no longer U2.5 (VBUS)
Other:
- note added: "EoS ESP32 DevKit, rev A. Designed by Kartikeydheer Srivastava. Copyright (c) 2026 Kartikeydheer Srivastava. All rights reserved; see LICENSE.txt. Values from Espressif's ESP32-WROOM-32E datasheet v2.1 (sections 6 and 9) and ESP32 Hardware Design Guidelines, the esptool docs (automatic bootloader), Silicon Labs CP2102N Rev. 1.5, Diodes AP7361C DS37274, onsemi MMBT3904, Nexperia PMEG6010CEH, Littel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"
- note removed: "EoS ESP32 DevKit, rev A. Designed by Kartikeydheer Srivastava. Copyright (c) 2026 Kartikeydheer Srivastava. All rights reserved; see LICENSE.txt. Values from Espressif's ESP32-WROOM-32E datasheet v2.1 (sections 6 and 9) and ESP32 Hardware Design Guidelines, the esptool docs (automatic bootloader), Silicon Labs CP2102N Rev. 1.5, Diodes AP7361C DS37274, onsemi MMBT3904, Nexperia PMEG6010CEH, ST USB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"
Changed lines of the file:
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@@
 	)
 	(symbol
-		(lib_id "Power_Protection:USBLC6-2SC6")
+		(lib_id "Power_Protection:SP0503BAHT")
 		(at 129.54 110.49 0)
 		(unit 1)
@@
 		(dnp no)
 		(property "Reference" "U2"
-			(at 129.54 104.14 0)
+			(at 134.62 107.95 0)
 			(effects
 				(font
@@
 			)
 		)
-		(property "Value" "USBLC6-2SC6"
-			(at 129.54 106.68 0)
+		(property "Value" "SP0503BAHTG"
+			(at 134.62 109.22 0)
 			(effects
 				(font
@@
 			)
 		)
-		(property "Footprint" "Package_TO_SOT_SMD:SOT-23-6"
-			(at 130.81 116.84 0)
+		(property "Footprint" "Package_TO_SOT_SMD:SOT-143"
+			(at 134.62 111.76 0)
 			(effects
 				(font
@@
 			)
 		)
-		(property "Datasheet" "https://www.st.com/resource/en/datasheet/usblc6-2.pdf"
-			(at 130.81 118.11 0)
+		(property "Datasheet" "http://www.littelfuse.com/~/media/files/littelfuse/technical%20resources/documents/data%20sheets/sp05xxba.pdf"
+			(at 132.08 106.68 0)
 			(effects
 				(font
@@
 			)
 		)
-		(property "Description" "Very low capacitance ESD protection diode, 2 data-line, SOT-23-6"
+		(property "Description" "TVS Diode Array, 5.5V Standoff, 3 Channels, SOT-143 package"
 			(at 129.54 110.49 0)
 			(effects
@@
 			)
 		)
-		(property "Manufacturer" "STMicroelectronics"
+		(property "Manufacturer" "Littelfuse"
 			(at 129.54 110.49 0)
 			(effects
@@
 			)
 		)
-		(property "MPN" "USBLC6-2SC6"
+		(property "MPN" "SP0503BAHTG"
 			(at 129.54 110.49 0)
 			(effects
@@
 			)
 		)
-		(property "Description" "USB ESD protection, D+/D- and VBUS (ST DS4260 Rev. 7)"
+		(property "Description" "USB ESD protection, three diodes to GND on D+, D- and VBUS, no path between them (CP2102N data sheet Figure 2.5)"
 			(at 129.54 110.49 0)
 			(effects
@@
 		(pin "4"
 		)
-		(pin "5"
-		)
-		(pin "6"
-		)
 		(instances
 			(project "eos-esp32-devkit"
@@
 	(wire
 		(pts
-			(xy 124.46 110.49)
-			(xy 121.92 110.49)
-		)
-		(stroke
-			(width 0)
-			(type default)
-		)
-	)
-	(label "USB_D+"
-		(at 121.92 110.49 180)
-		(fields_autoplaced yes)
-		(effects
-			(font
-				(size 1.27 1.27)
-			)
-			(justify right bottom)
-		)
-	)
-	(wire
-		(pts
-			(xy 134.62 110.49)
-			(xy 137.16 110.49)
-		)
-		(stroke
-			(width 0)
-			(type default)
-		)
-	)
-	(label "USB_D+"
-		(at 137.16 110.49 0)
-		(fields_autoplaced yes)
-		(effects
-			(font
-				(size 1.27 1.27)
-			)
-			(justify left bottom)
-		)
-	)
-	(wire
-		(pts
-			(xy 124.46 113.03)
-			(xy 121.92 113.03)
+			(xy 129.54 115.57)
+			(xy 129.54 118.11)
 		)
 		(stroke
@@
 		)
 	)
-	(label "USB_D-"
-		(at 121.92 113.03 180)
+	(label "GND"
+		(at 129.54 118.11 270)
 		(fields_autoplaced yes)
 		(effects
@@
 	(wire
 		(pts
-			(xy 134.62 113.03)
-			(xy 137.16 113.03)
+			(xy 127 105.41)
+			(xy 127 102.87)
 		)
 		(stroke
@@
 	)
 	(label "USB_D-"
-		(at 137.16 113.03 0)
+		(at 127 102.87 90)
 		(fields_autoplaced yes)
 		(effects
@@
 	(wire
 		(pts
-			(xy 129.54 118.11)
-			(xy 129.54 120.65)
+			(xy 129.54 105.41)
+			(xy 129.54 102.87)
 		)
 		(stroke
@@
 		)
 	)
-	(label "GND"
-		(at 129.54 120.65 270)
+	(label "USB_D+"
+		(at 129.54 102.87 90)
 		(fields_autoplaced yes)
 		(effects
@@
 				(size 1.27 1.27)
 			)
-			(justify right bottom)
+			(justify left bottom)
 		)
 	)
 	(wire
 		(pts
-			(xy 129.54 105.41)
-			(xy 129.54 102.87)
+			(xy 132.08 105.41)
+			(xy 132.08 102.87)
 		)
 		(stroke
@@
 	)
 	(label "VBUS"
-		(at 129.54 102.87 90)
+		(at 132.08 102.87 90)
 		(fields_autoplaced yes)
 		(effects
@@
 		)
 	)
-	(text "EoS ESP32 DevKit, rev A. Designed by Kartikeydheer Srivastava.\nCopyright (c) 2026 Kartikeydheer Srivastava. All rights reserved; see LICENSE.txt.\nValues from Espressif's ESP32-WROOM-32E datasheet v2.1 (sections 6 and 9) and ESP32 Hardware\nDesign Guidelines, the esptool docs (automatic bootloader), Silicon Labs CP2102N Rev. 1.5,\nDiodes AP7361C DS37274, onsemi MMBT3904, Nexperia PMEG6010CEH, ST USBLC6-2, Littelfuse 1206L, Kingbright.\nU1: KiCad's ESP32-WROOM-32E symbol; its stacked GND pin [1,15,38,39] is expanded to the four pads.\nR12 (5.1 kohm) bleeds D1's reverse leakage off VBUS, so a 5V-pin supply does not fake a USB host.\nGPIO6-11 are the module's internal flash pins and are not led out: J2 16-18, J3 17-19 are NC.\nHeader grid and pinout from Espressif's DevKitC V4 user guide (positions and names only)."
+	(text "EoS ESP32 DevKit, rev A. Designed by Kartikeydheer Srivastava.\nCopyright (c) 2026 Kartikeydheer Srivastava. All rights reserved; see LICENSE.txt.\nValues from Espressif's ESP32-WROOM-32E datasheet v2.1 (sections 6 and 9) and ESP32 Hardware\nDesign Guidelines, the esptool docs (automatic bootloader), Silicon Labs CP2102N Rev. 1.5,\nDiodes AP7361C DS37274, onsemi MMBT3904, Nexperia PMEG6010CEH, Littelfuse SP0503BAHTG, Littelfuse 1206L, Kingbright.\nU1: KiCad's ESP32-WROOM-32E symbol; its stacked GND pin [1,15,38,39] is expanded to the four pads.\nR12 (5.1 kohm) bleeds D1's reverse leakage off VBUS, so a 5V-pin supply does not fake a USB host.\nGPIO6-11 are the module's internal flash pins and are not led out: J2 16-18, J3 17-19 are NC.\nHeader grid and pinout from Espressif's DevKitC V4 user guide (positions and names only)."
 		(exclude_from_sim no)
 		(at 330 330 0)
