File: boards/eos/eos-lpc55s69-board/hardware/eos-lpc55s69-board.kicad_pcb (KiCad board)
At the start: 4 copper layers, 68.6 x 53.3 mm, 99 parts, among them J1 USB-C, J2 USB-C, J3 Cortex Debug, J4 D8-SCL, J5 D0-D7, J6 POWER, J7 A0-A5, Q1 BSS138BK, Q2 BSS138BK, Q3 BSS138BK, SW1 RESET, SW2 ISP, SW3 USER, U1 SP0503BAHTG, U2 SP0503BAHTG, U3 TPS2116, U4 TPS7A91, U5 CP2102N-A02-GQFN24, U6 LPC55S69JBD100, Y1 16MHz, Y2 32.768kHz

Commit message: fix(boards): rebuild the ten boards made before the no-via-in-pad rule (#55)
PR #64's generator keeps vias out of surface pads (a chip's exposed pad
aside) and 0.1 mm from their own net's pads. Ten boards on master were built
before that rule and had 34 pads with a via in or beside them. They are
rebuilt with the same generator: ATmega328P, RA2E1, KE16Z, KL25, STM32 64,
ESP32 DevKit, Learn RP2350, LPC55S69, CM4 Base and CM5 Base. Each builds at
ERC 0, DRC errors 0, unconnected 0 and parity 0, with the same parts, values,
nets and positions and the same DRC warnings as before.

Where the router could no longer close a short link without a via in a pad,
or left a ground pad without a good path to a via, the design files use
routing options only: priority routes, fanout_first, ground_vias, and a
bottom-layer router keep-out under KL25's crystal (so RESET_b no longer runs
under it). ViaInPadTest drops BUILT_BEFORE_THE_RULE; it now allows only Learn
RP2350's two Raspberry Pi reference vias, named by position. READMEs, TASKS
and CHANGELOG follow the rebuilt copper. Independent verification: three
rounds; the owner adopted a two-layer pour-island criterion (TASKS.md).

Part of #55.
Routing:
- net /RESETN: track 98.2 -> 82.0 mm, vias 1 -> 0
- net /LED_R: track 32.3 -> 45.1 mm, vias 0 -> 2
- net +5V: track 66.5 -> 58.3 mm
- net /SWDIO: track 24.2 -> 30.2 mm
- net /A3: track 32.3 -> 27.2 mm
- net /SWO: track 25.3 -> 30.2 mm, vias 2 -> 0
- net /VDDA: track 17.2 -> 12.9 mm, vias 2 -> 0
- net /ISP_N: track 42.9 -> 46.3 mm
- net /SWCLK: track 23.0 -> 20.2 mm
- net /RGB_RK: track 11.2 -> 8.78 mm
- net /USER_BTN: track 38.5 -> 36.4 mm
- net /RGB_RD: track 6.55 -> 8.23 mm, vias 2 -> 0
- net /LED_G: track 33.5 -> 31.9 mm
- net /A4: track 31.1 -> 29.7 mm
- net /MUX_PR1: track 3.59 -> 4.74 mm, vias 2 -> 0
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