File: boards/eos/eos-stm32-64/hardware/eos-stm32-64.kicad_pcb (KiCad board)
At the start: 2 copper layers, 70 x 82.5 mm, 99 parts, among them CN10 CN10, CN5 D8-D15, CN6 POWER, CN7 CN7, CN8 ANALOG, CN9 D0-D7, J1 USB-C, J2 USB-C, J3 Cortex Debug, J4 IDD, U1 STM32F411RET6, U2 CP2102N-A02-GQFN20, U3 AP7361C-33, U4 AP63205, U5 SP0503BAHTG, U6 SP0503BAHTG, Y1 8MHz, Y2 32.768kHz

Commit message: fix(boards): rebuild the ten boards made before the no-via-in-pad rule (#55)
PR #64's generator keeps vias out of surface pads (a chip's exposed pad
aside) and 0.1 mm from their own net's pads. Ten boards on master were built
before that rule and had 34 pads with a via in or beside them. They are
rebuilt with the same generator: ATmega328P, RA2E1, KE16Z, KL25, STM32 64,
ESP32 DevKit, Learn RP2350, LPC55S69, CM4 Base and CM5 Base. Each builds at
ERC 0, DRC errors 0, unconnected 0 and parity 0, with the same parts, values,
nets and positions and the same DRC warnings as before.

Where the router could no longer close a short link without a via in a pad,
or left a ground pad without a good path to a via, the design files use
routing options only: priority routes, fanout_first, ground_vias, and a
bottom-layer router keep-out under KL25's crystal (so RESET_b no longer runs
under it). ViaInPadTest drops BUILT_BEFORE_THE_RULE; it now allows only Learn
RP2350's two Raspberry Pi reference vias, named by position. READMEs, TASKS
and CHANGELOG follow the rebuilt copper. Independent verification: three
rounds; the owner adopted a two-layer pour-island criterion (TASKS.md).

Part of #55.
Routing:
- net GND: track 517.4 -> 474.5 mm, vias 102 -> 91
- net /PB5: track 87.2 -> 53.2 mm, vias 2 -> 1
- net /PA15: track 88.1 -> 116.6 mm, vias 1 -> 4
- net /PA2: track 127.0 -> 101.6 mm, vias 2 -> 4
- net /PA13: track 105.3 -> 130.3 mm, vias 3 -> 2
- net /VBAT: track 57.3 -> 78.6 mm, vias 2 -> 0
- net /PA3: track 127.8 -> 107.4 mm, vias 2 -> 4
- net /BOOT0: track 82.2 -> 101.0 mm, vias 2 -> 3
- net /VDD_MCU: track 161.9 -> 177.7 mm, vias 6 -> 11
- net /USB_DP: track 66.3 -> 51.4 mm
- net /PA14: track 85.7 -> 98.2 mm, vias 1 -> 2
- net /PA12_HDR: track 34.1 -> 22.4 mm
- net /PB15: track 39.4 -> 29.2 mm, vias 1 -> 0
- net /PC6: track 34.6 -> 44.8 mm, vias 0 -> 1
- net /PB13: track 43.1 -> 33.2 mm, vias 1 -> 0
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